Commit message: Simulation sensors and sub to cmd_vel

File: src/rover_description/urdf/rover_base.urdf (robot description, URDF)
Before this commit: robot rover, 10 links, 9 joints
Links:
- added link gps_link, mass 0.05; collision box size=0.05 0.05 0.02; visual box size=0.05 0.05 0.02
- added link imu_link, mass 0.01; collision box size=0.03 0.03 0.01; visual box size=0.03 0.03 0.01
- added link lidar_link, mass 0.263893782901543; collision mesh filename=package://rover_description/meshes/lidar.STL; visual mesh filename=package://rover_description/meshes/lidar.STL
Joints:
- added joint gps_joint: type fixed, parent base_link, child gps_link, origin xyz=0 0 0.05 rpy=0 0 0
- added joint imu_joint: type fixed, parent base_link, child imu_link, origin xyz=0 0 0 rpy=0 0 0
- added joint lidar_joint: type fixed, parent base_link, child lidar_link, origin xyz=0.2 0 0.2 rpy=-0.3 0 -1.5708

Commit message: adjusting cameras for CV

File: src/rover_description/urdf/rover_base.urdf (robot description, URDF)
Before this commit: robot rover, 13 links, 12 joints
Joints:
- joint LCam_joint: origin xyz=-0.025966 0.078001 0.2496 rpy=0 0 0 -> xyz=-0.025966 ${camera_baseline_half} 0.275 rpy=0 0 0.3491
- joint RCam_joint: origin xyz=-0.025966 -0.078591 0.2496 rpy=0 0 0 -> xyz=-0.025966 -${camera_baseline_half} 0.275 rpy=0 0 -0.3491
