Commit message: Manual Working, lidar and wheels movement configured

File: src/rover26/description/sensors/lidar.xacro (robot description, xacro)
@@ -12,7 +12,6 @@
     <parent link="base_link"/>
     <child link="lidar_link"/>
-    <!-- old xyz="-0.0014001 -0.27365 0.04"
-         new xyz=" 0.27365  -0.0014001 0.04" -->
-    <origin xyz="0.27365 -0.0014001 0.04" rpy="0 0 0"/>
+    <!-- <origin xyz="0.27365 -0.0014001 0.04" rpy="0 0 0"/> lidar is now rotated 180 degrees-->
+    <origin xyz="0.27365 -0.0014001 0.04" rpy="0 0 3.14159"/>
   </joint>
   <!-- ═══════════════════════════════════════════════════════════════════════
