Commit message: Some Autonomus Adjusments. New Odometry

File: src/rover26/description/sensors/lidar.xacro (robot description, xacro)
@@ -13,5 +13,5 @@
     <child link="lidar_link"/>
     <!-- <origin xyz="0.27365 -0.0014001 0.04" rpy="0 0 0"/> lidar is now rotated 180 degrees-->
-    <origin xyz="0.27365 -0.0014001 0.04" rpy="0 0 3.14159"/>
+    <origin xyz="0.0 -0.00140010000 0.04" rpy="0 0 3.14159"/>
   </joint>
   <!-- ═══════════════════════════════════════════════════════════════════════
@@ -55,6 +55,6 @@
         </scan>
         <range>
-          <min>0.3</min>
-          <max>25.0</max>
+          <min>0.5</min>
+          <max>100.0</max>
           <resolution>0.01</resolution>
         </range>

Commit message: Lande detection and point publisher changes

File: src/rover26/description/sensors/lidar.xacro (robot description, xacro)
@@ -13,5 +13,5 @@
     <child link="lidar_link"/>
     <!-- <origin xyz="0.27365 -0.0014001 0.04" rpy="0 0 0"/> lidar is now rotated 180 degrees-->
-    <origin xyz="0.0 -0.00140010000 0.04" rpy="0 0 3.14159"/>
+    <origin xyz="0.085 -0.0 0.20" rpy="0 0 3.14159"/>
   </joint>
   <!-- ═══════════════════════════════════════════════════════════════════════
